File: Adafruit MPR121 Capacitive Touch Shield Original.sch (EAGLE design)
At the start: 52 parts, among them Q1 BSS138, Q2 BSS138, SW2 6mm tact, U2 MPR121, U4 AP2127K-3.3

Commit message: Add updated board files.
Parts:
- removed SJ1: (no value), microbuilder:SOLDERJUMPER_2WAY
- AL1, AL10, AL11, AL12, AL2, AL3, AL4, AL5, AL6, AL7, AL8, AL9: device adafruit_electromech:ALLIGATORCLIP_MICRO -> microbuilder:ALLIGATORCLIP_MICRO
- FID1, FID2, FID3: value FIDUCIAL_1MM -> FIDUCIAL""; device microbuilder:FIDUCIAL_1MM -> microbuilder:FIDUCIAL""
- SW2: value 6mm tact -> SPST_TACT-EVQQ2; device adafruit_electromech:SWITCH_TACT_SMT_6MM -> adafruit:SPST_TACT-EVQQ2
- U$41: value ARDUINO_R3_ICSP_NODIM -> ARDUINO_R3_ICSP; device adafruit:ARDUINO_R3_ICSP_NODIM -> adafruit:ARDUINO_R3_ICSP
- U2: device adafruit_sensor:MPR121Q -> microbuilder:MPR121Q
- U4: value AP2127K-3.3 -> MIC5225-3.3; device adafruit_power:VREG_SOT23-5 -> microbuilder:VREG_SOT23-5
Connections:
- removed net VCCIO: JP4.7, R2.2, R4.2, SJ1.2, U$41.IOREF
- new net IORESET: JP4.7, U$41.IOREF
- net +5V: now also R2.2, R4.2; no longer SJ1.1
- net 3.3V: no longer SJ1.3
